Commit message: Fix Python venv CMake interference; suppress empty calib_file xacro warning
CMakeLists.txt: set Python3_FIND_VIRTUALENV STANDARD before
find_package(ament_cmake) so CMake falls back to system Python
when a broken or absent virtualenv is active in the environment.

config/bno055.urdf.xacro: capture calib_file arg in a xacro:property
and wrap the <param> in <xacro:if> so it is only emitted when a path
is actually provided, suppressing the ros2_control 'text not specified
in the calib_file tag' warning on default (empty) launches.

File: config/bno055.urdf.xacro (robot description, xacro)
@@ -7,4 +7,5 @@
   <xacro:arg name="enable_mock" default="false"/>
   <xacro:arg name="calib_file"  default=""/>          <!-- Path to calibration YAML file (empty = uncalibrated startup) -->
+  <xacro:property name="calib_file_path" value="$(arg calib_file)"/>
   <!-- Robot links -->
   <link name="base_link"/>
@@ -33,5 +34,7 @@
       <param name="axis_remap">$(arg axis_remap)</param>     <!-- Axis placement config: P0-P7 (default: P1) -->
       <param name="enable_mock">$(arg enable_mock)</param>   <!-- Simulation mode, no hardware required (default: false) -->
-      <param name="calib_file">$(arg calib_file)</param>       <!-- Path to calibration YAML saved by bno055_calib_node (empty = none) -->
+      <xacro:if value="${calib_file_path != ''}">             <!-- Only emitted when a path is provided -->
+        <param name="calib_file">${calib_file_path}</param>
+      </xacro:if>
     </hardware>
     <sensor name="bno055">
